File: 881.kicad_pcb (KiCad board)
At the start: 4 copper layers, 38 x 105 mm, 114 parts, among them J1 RUN/STOP, J10 RS IN, J11 CP IN, J12 MA IN, J13 CB IN, J14 CY IN, J15 OH IN, J16 CH IN, J2 SYNC24 CLK, J3 ASSIGN 1, J4 ASSIGN 2, J5 BD IN, J6 SD IN, J7 LT IN, J8 MT IN, J9 HT IN, P1 CONN_02X03, Q1 MMBT3904, Q10 MMBT3904, Q11 MMBT3904, Q12 MMBT3904, Q13 MMBT3904, Q14 MMBT3906, Q2 MMBT3904, Q3 MMBT3904, Q4 MMBT3904, Q5 MMBT3904, Q6 MMBT3904, Q7 MMBT3904, Q8 MMBT3904, Q9 MMBT3904, U1 74HC165, U2 74HC165, U7 74AHCT1G125GW, X1 MIDI OUT, X2 SYNC24

Commit message: 2024 update with panel
Parts:
- removed D17: LED, LEDs:LED_0805
- removed Q13: MMBT3904, MyModules:SOT23-132-JRL
- removed R47: 1K, MyModules:SM0603-R-YAGEO
- removed R48: 10K, MyModules:SM0603-R-YAGEO
- added G***: LOGO, LOGO, B.Cu at (120.2, 61.0)
- R49: value 1K -> 2.7K
Connections:
- R46 pad 1: Net-(Q13-Pad1) -> Net-(C4-Pad1)
Routing:
- net Net-(C4-Pad1): track 3.69 -> 9.76 mm
- net Net-(Q13-Pad3): track 3.93 -> 0.00 mm
- net Net-(D18-Pad1): track 6.44 -> 3.28 mm
- net Net-(D18-Pad2): track 6.46 -> 4.43 mm
- net Net-(Q13-Pad1): track 1.52 -> 0.00 mm
- net +5V: track 43.7 -> 42.6 mm, vias 29 -> 28
Other:
- board text added: "r2.1 01/2021"
- board text removed: "881"
- board text removed: "r2.0 10/2020"
